File: board/ttpcb.sch (EAGLE design)
At the start: 9 parts

Commit message: u1
Parts:
- U$1, U$3, U$4, U$5, U$6, U$7, U$8, U$9: value QRE1113QRE1113GR-3D -> QRE1113QRE1113GR; device TinyTony_ShenzenReady:QRE1113QRE1113GR-3D -> TinyTony_ShenzenReady:QRE1113QRE1113GR
